File: jacdac_EC30_20x20_template.kicad_pcb (KiCad board)
At the start: 2 copper layers, 25 x 25 mm, 6 parts

Commit message: Moved LED position, added component keepouts
Parts:
- MH3: value Val** -> jacdac_hole_PWR_MH3
